File: PCB/Weather-Station.sch (KiCad schematic (older format))
At the start: 47 parts, among them J1 Biruta, J10 Conn_01x02, J11 Conn_01x02, J12 Conn_01x02, J13 Conn_01x02, J14 Conn_01x02, J15 Conn_01x02, J2 Power, J3 DataLogger, J4 BME280, J5 Pluviometro, J6 Anemometro, J7 FTDI, J8 Conn_01x02, J9 Conn_01x02, SW1 SW_Push_SPDT, SW2 SW_Push, SW3 SW_SPDT, U1 AP1117-33, U2 ESP-32S, U3 AP1117-33, U4 ADS1115, U5 ADS1115, U6 ADS1115, U7 ADS1115

Commit message: Fazendo pcb
Signed-off-by: Gustavo Costa <gustavocosta@ic.ufal.br>
Parts:
- added R10, R9: 10k, Resistors_SMD:R_0805, symbol R
Connections:
- net SCL: now also R9.2
- net SDA: now also R10.2
- net at U4.4 (AIN0): now also J8.1 (Pin_1); no longer J8.2 (Pin_2)
- net at U4.5 (AIN1): now also J8.2 (Pin_2); no longer J8.1 (Pin_1)
- net at U4.6 (AIN2): now also J9.1 (Pin_1); no longer J9.2 (Pin_2)
- net at U4.7 (AIN3): now also J9.2 (Pin_2); no longer J9.1 (Pin_1)
- net at U5.4 (AIN0): now also J10.1 (Pin_1); no longer J10.2 (Pin_2)
- net at U5.5 (AIN1): now also J10.2 (Pin_2); no longer J10.1 (Pin_1)
- net at U5.6 (AIN2): now also J11.1 (Pin_1); no longer J11.2 (Pin_2)
- net at U5.7 (AIN3): now also J11.2 (Pin_2); no longer J11.1 (Pin_1)
- net at U6.4 (AIN0): now also J12.1 (Pin_1); no longer J12.2 (Pin_2)
- net at U6.5 (AIN1): now also J12.2 (Pin_2); no longer J12.1 (Pin_1)
- net at U6.6 (AIN2): now also J13.1 (Pin_1); no longer J13.2 (Pin_2)
- net at U6.7 (AIN3): now also J13.2 (Pin_2); no longer J13.1 (Pin_1)
- net at U7.4 (AIN0): now also J14.1 (Pin_1); no longer J14.2 (Pin_2)
- net at U7.5 (AIN1): now also J14.2 (Pin_2); no longer J14.1 (Pin_1)
- net at U7.6 (AIN2): now also J15.1 (Pin_1); no longer J15.2 (Pin_2)
- net at U7.7 (AIN3): now also J15.2 (Pin_2); no longer J15.1 (Pin_1)
- new net: R10.1, R9.1

Commit message: Finalizando PCB
Signed-off-by: Gustavo <gustavocosta@ic.ufal.br>
Connections:
- net +5V: now also R10.1, R9.1
Changed lines of the file:
@@
-	1    0    0    -1
-$EndComp
-$Comp
-L ADS1115 U4
-U 1 1 5B8947BB
-P 2550 5900
-F 0 "U4" H 2550 5400 60  0000 C CNN
-F 1 "ADS1115" H 2550 6400 60  0000 C CNN
-F 2 "Housings_SSOP:MSOP-10_3x3mm_Pitch0.5mm" H 2500 6000 60  0001 C CNN
-F 3 "" H 2500 6000 60  0001 C CNN
-	1    2550 5900
-	1    0    0    -1
-$EndComp
-$Comp
-L ADS1115 U5
-U 1 1 5B8948D4
-P 4500 5900
-F 0 "U5" H 4500 5400 60  0000 C CNN
-F 1 "ADS1115" H 4500 6400 60  0000 C CNN
-F 2 "Housings_SSOP:MSOP-10_3x3mm_Pitch0.5mm" H 4450 6000 60  0001 C CNN
-F 3 "" H 4450 6000 60  0001 C CNN
-	1    4500 5900
-	1    0    0    -1
-$EndComp
-$Comp
-L ADS1115 U6
-U 1 1 5B89494D
-P 6400 5900
-F 0 "U6" H 6400 5400 60  0000 C CNN
-F 1 "ADS1115" H 6400 6400 60  0000 C CNN
-F 2 "Housings_SSOP:MSOP-10_3x3mm_Pitch0.5mm" H 6350 6000 60  0001 C CNN
-F 3 "" H 6350 6000 60  0001 C CNN
-	1    6400 5900
-	1    0    0    -1
-$EndComp
-$Comp
-L ADS1115 U7
-U 1 1 5B894A7A
-P 8400 5900
-F 0 "U7" H 8400 5400 60  0000 C CNN
-F 1 "ADS1115" H 8400 6400 60  0000 C CNN
-F 2 "Housings_SSOP:MSOP-10_3x3mm_Pitch0.5mm" H 8350 6000 60  0001 C CNN
-F 3 "" H 8350 6000 60  0001 C CNN
-	1    8400 5900
 	1    0    0    -1
 $EndComp
@@
 Wire Wire Line
 	2700 4550 2700 4600
+$Comp
+L ADS1115 U7
+U 1 1 5B894A7A
+P 8400 5900
+F 0 "U7" H 8400 5400 60  0000 C CNN
+F 1 "ADS1115" H 8400 6400 60  0000 C CNN
+F 2 "Housings_SSOP:MSOP-10_3x3mm_Pitch0.5mm" H 8350 6000 60  0001 C CNN
+F 3 "" H 8350 6000 60  0001 C CNN
+	1    8400 5900
+	1    0    0    -1
+$EndComp
+$Comp
+L ADS1115 U6
+U 1 1 5B89494D
+P 6400 5900
+F 0 "U6" H 6400 5400 60  0000 C CNN
+F 1 "ADS1115" H 6400 6400 60  0000 C CNN
+F 2 "Housings_SSOP:MSOP-10_3x3mm_Pitch0.5mm" H 6350 6000 60  0001 C CNN
+F 3 "" H 6350 6000 60  0001 C CNN
+	1    6400 5900
+	1    0    0    -1
+$EndComp
+$Comp
+L ADS1115 U5
+U 1 1 5B8948D4
+P 4500 5900
+F 0 "U5" H 4500 5400 60  0000 C CNN
+F 1 "ADS1115" H 4500 6400 60  0000 C CNN
+F 2 "Housings_SSOP:MSOP-10_3x3mm_Pitch0.5mm" H 4450 6000 60  0001 C CNN
+F 3 "" H 4450 6000 60  0001 C CNN
+	1    4500 5900
+	1    0    0    -1
+$EndComp
+$Comp
+L ADS1115 U4
+U 1 1 5B8947BB
+P 2550 5900
+F 0 "U4" H 2550 5400 60  0000 C CNN
+F 1 "ADS1115" H 2550 6400 60  0000 C CNN
+F 2 "Housings_SSOP:MSOP-10_3x3mm_Pitch0.5mm" H 2500 6000 60  0001 C CNN
+F 3 "" H 2500 6000 60  0001 C CNN
+	1    2550 5900
+	1    0    0    -1
+$EndComp
+Wire Wire Line
+	2500 4500 2500 4550
+Connection ~ 2500 4550
 $EndSCHEMATC
