File: PCB/Weather-Station.kicad_pcb (KiCad board)
At the start: 2 copper layers, 65 x 60 mm, 49 parts, among them J1 Biruta, J10 Conn_01x02, J11 Conn_01x02, J12 Conn_01x02, J13 Conn_01x02, J14 Conn_01x02, J15 Conn_01x02, J2 Power, J3 DataLogger, J4 BME280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

Commit message: Ajustando PCB
Signed-off-by: Gustavo Costa <gustavocosta@ic.ufal.br>
Routing:
- net GND: track 77.2 -> 75.5 mm
Other:
- outline, holes or cut-outs redrawn
Changed lines of the file:
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@@
-(kicad_pcb (version 4) (host pcbnew 4.0.7)
+(kicad_pcb (version 4) (host pcbnew 4.0.7-e2-6376~58~ubuntu16.04.1)
   (general
     (links 121)
@@
     (area 122.424999 49.924999 187.575001 110.075001)
     (thickness 1.6)
-    (drawings 10)
-    (tracks 421)
+    (drawings 14)
+    (tracks 423)
     (zones 0)
     (modules 49)
@@
     )
   )
+  (gr_arc (start 186.5 109) (end 187.5 109) (angle 90) (layer Edge.Cuts) (width 0.15))
+  (gr_arc (start 186.5 51) (end 186.5 50) (angle 90) (layer Edge.Cuts) (width 0.15))
+  (gr_arc (start 123.5 51) (end 122.5 51) (angle 90) (layer Edge.Cuts) (width 0.15))
+  (gr_arc (start 123.5 109) (end 123.5 110) (angle 90) (layer Edge.Cuts) (width 0.15))
   (gr_line (start 154.5 74.5) (end 187.5 74.5) (layer Margin) (width 0.2))
   (gr_line (start 154.5 110) (end 154.5 74.5) (layer Margin) (width 0.2))
@@
     (arrow2b (pts (xy 122.5 40.25) (xy 123.626504 39.663579)))
   )
-  (gr_line (start 187.5 50) (end 122.5 50) (layer Edge.Cuts) (width 0.15))
-  (gr_line (start 187.5 110) (end 187.5 50) (layer Edge.Cuts) (width 0.15))
-  (gr_line (start 122.5 110) (end 187.5 110) (layer Edge.Cuts) (width 0.15))
-  (gr_line (start 122.5 50) (end 122.5 110) (layer Edge.Cuts) (width 0.15))
+  (gr_line (start 186.5 50) (end 123.5 50) (layer Edge.Cuts) (width 0.15))
+  (gr_line (start 187.5 109) (end 187.5 51) (layer Edge.Cuts) (width 0.15))
+  (gr_line (start 123.5 110) (end 186.5 110) (layer Edge.Cuts) (width 0.15))
+  (gr_line (start 122.5 51) (end 122.5 109) (layer Edge.Cuts) (width 0.15))
+  (segment (start 166.45 63) (end 166.45 68) (width 0.3) (layer F.Cu) (net 1))
   (segment (start 167.684446 65.255554) (end 168.2 64.74) (width 0.3) (layer F.Cu) (net 1))
   (segment (start 167.684446 68.712802) (end 167.684446 65.255554) (width 0.3) (layer F.Cu) (net 1))
@@
   (segment (start 126.25 80.2) (end 156.197248 80.2) (width 0.3) (layer F.Cu) (net 1))
   (segment (start 168.2 64.74) (end 167.8 65.14) (width 0.3) (layer F.Cu) (net 1))
-  (segment (start 166.45 63) (end 166.45 68) (width 0.3) (layer F.Cu) (net 1))
   (segment (start 173.2 59.74) (end 169.41 59.74) (width 0.3) (layer F.Cu) (net 1))
   (segment (start 166.45 62.7) (end 166.45 63) (width 0.3) (layer F.Cu) (net 1))
@@
   (segment (start 176.11 59.74) (end 178.75 57.1) (width 0.3) (layer F.Cu) (net 1))
   (segment (start 178.75 57.1) (end 178.75 56.45) (width 0.3) (layer F.Cu) (net 1))
+  (segment (start 164.63 78.73073) (end 164.628356 78.732374) (width 0.3) (layer B.Cu) (net 2))
+  (segment (start 164.63 76.5) (end 164.63 78.73073) (width 0.3) (layer B.Cu) (net 2))
+  (via (at 164.628356 78.732374) (size 0.52) (drill 0.335) (layers F.Cu B.Cu) (net 2))
+  (segment (start 164.63 74.389427) (end 164.628356 74.387783) (width 0.3) (layer F.Cu) (net 2))
+  (segment (start 164.63 76.5) (end 164.63 74.389427) (width 0.3) (layer F.Cu) (net 2))
+  (via (at 164.628356 74.387783) (size 0.52) (drill 0.335) (layers F.Cu B.Cu) (net 2))
   (segment (start 145.3 96) (end 146.699911 96) (width 0.3) (layer F.Cu) (net 2))
   (segment (start 146.699911 96) (end 147.178959 96.479048) (width 0.3) (layer F.Cu) (net 2))
@@
   (segment (start 184 62.12) (end 185.413492 62.12) (width 0.3) (layer F.Cu) (net 2))
   (segment (start 185.413492 62.12) (end 185.543492 62.25) (width 0.3) (layer F.Cu) (net 2))
-  (segment (start 164.63 76.5) (end 164.63 78.62) (width 0.3) (layer B.Cu) (net 2))
-  (segment (start 164.63 78.62) (end 164.5 78.75) (width 0.3) (layer B.Cu) (net 2))
-  (via (at 164.5 78.75) (size 0.52) (drill 0.335) (layers F.Cu B.Cu) (net 2))
-  (segment (start 164.63 76.5) (end 164.63 75.12) (width 0.3) (layer F.Cu) (net 2))
-  (segment (start 164.63 75.12) (end 166.25 73.5) (width 0.3) (layer F.Cu) (net 2))
-  (via (at 166.25 73.5) (size 0.52) (drill 0.335) (layers F.Cu B.Cu) (net 2))
   (segment (start 157.6 74.55) (end 159.45 74.55) (width 0.3) (layer F.Cu) (net 2))
   (segment (start 159.45 74.55) (end 159.5 74.5) (width 0.3) (layer F.Cu) (net 2))
@@
   (segment (start 140.565 60.39) (end 141.375 60.39) (width 0.175) (layer F.Cu) (net 21))
   (segment (start 141.375 60.39) (end 142.8 60.39) (width 0.175) (layer F.Cu) (net 21))
+  (segment (start 175.712145 65.792085) (end 175.458146 65.538086) (width 0.175) (layer F.Cu) (net 22))
+  (segment (start 179.87 69.94994) (end 175.712145 65.792085) (width 0.175) (layer F.Cu) (net 22))
+  (segment (start 179.87 76.5) (end 179.87 69.94994) (width 0.175) (layer F.Cu) (net 22))
+  (segment (start 174.12006 64.2) (end 175.204147 65.284087) (width 0.175) (layer B.Cu) (net 22))
+  (segment (start 175.204147 65.284087) (end 175.458146 65.538086) (width 0.175) (layer B.Cu) (net 22))
+  (segment (start 163.2 64.2) (end 174.12006 64.2) (width 0.175) (layer B.Cu) (net 22))
+  (via (at 175.458146 65.538086) (size 0.508) (drill 0.3302) (layers F.Cu B.Cu) (net 22))
   (segment (start 163.2 64.2) (end 160.8 64.2) (width 0.175) (layer F.Cu) (net 22))
-  (segment (start 173.2 64.2) (end 163.2 64.2) (width 0.175) (layer B.Cu) (net 22))
   (via (at 163.2 64.2) (size 0.508) (drill 0.3302) (layers F.Cu B.Cu) (net 22))
-  (segment (start 179.87 70.07) (end 174 64.2) (width 0.175) (layer F.Cu) (net 22))
-  (segment (start 174 64.2) (end 173.2 64.2) (width 0.175) (layer F.Cu) (net 22))
-  (via (at 173.2 64.2) (size 0.508) (drill 0.3302) (layers F.Cu B.Cu) (net 22))
-  (segment (start 179.87 76.5) (end 179.87 70.07) (width 0.175) (layer F.Cu) (net 22))
   (segment (start 163 52.8) (end 163 59.6) (width 0.175) (layer B.Cu) (net 23))
   (segment (start 163 59.6) (end 164.516661 61.116661) (width 0.175) (layer B.Cu) (net 23))
@@
   (segment (start 162.97 52.77) (end 163 52.8) (width 0.175) (layer F.Cu) (net 23))
   (via (at 163 52.8) (size 0.508) (drill 0.3302) (layers F.Cu B.Cu) (net 23))
+  (segment (start 173.685777 64.969287) (end 166.123862 64.969287) (width 0.175) (layer B.Cu) (net 24))
+  (segment (start 175.082237 66.365747) (end 173.685777 64.969287) (width 0.175) (layer B.Cu) (net 24))
   (segment (start 174.79 76.5) (end 175.082237 76.207763) (width 0.175) (layer B.Cu) (net 24))
-  (segment (start 175.082237 66.365747) (end 173.685777 64.969287) (width 0.175) (layer B.Cu) (net 24))
-  (segment (start 173.685777 64.969287) (end 166.123862 64.969287) (width 0.175) (layer B.Cu) (net 24))
+  (segment (start 165.764652 61.972209) (end 165.764652 64.610077) (width 0.175) (layer F.Cu) (net 24))
+  (segment (start 160.8 60.39) (end 164.182443 60.39) (width 0.175) (layer F.Cu) (net 24))
+  (via (at 165.764652 64.969287) (size 0.508) (drill 0.3302) (layers F.Cu B.Cu) (net 24))
+  (segment (start 166.123862 64.969287) (end 165.764652 64.969287) (width 0.175) (layer B.Cu) (net 24))
+  (segment (start 165.764652 64.610077) (end 165.764652 64.969287) (width 0.175) (layer F.Cu) (net 24))
   (segment (start 175.082237 76.207763) (end 175.082237 66.365747) (width 0.175) (layer B.Cu) (net 24))
-  (segment (start 166.123862 64.969287) (end 165.764652 64.969287) (width 0.175) (layer B.Cu) (net 24))
-  (segment (start 165.764652 62.319801) (end 165.764652 64.610077) (width 0.175) (layer F.Cu) (net 24))
-  (segment (start 163.834851 60.39) (end 165.764652 62.319801) (width 0.175) (layer F.Cu) (net 24))
-  (segment (start 160.8 60.39) (end 163.834851 60.39) (width 0.175) (layer F.Cu) (net 24))
-  (segment (start 165.764652 64.610077) (end 165.764652 64.969287) (width 0.175) (layer F.Cu) (net 24))
-  (via (at 165.764652 64.969287) (size 0.508) (drill 0.3302) (layers F.Cu B.Cu) (net 24))
+  (segment (start 164.182443 60.39) (end 165.764652 61.972209) (width 0.175) (layer F.Cu) (net 24))
   (segment (start 165.2 65.6) (end 167.227655 67.627655) (width 0.175) (layer B.Cu) (net 25))
+  (segment (start 167.227655 67.627655) (end 173.750931 67.627655) (width 0.175) (layer B.Cu) (net 25))
+  (segment (start 174.645092 74.104908) (end 173.099999 75.650001) (width 0.175) (layer B.Cu) (net 25))
   (segment (start 174.645092 68.521816) (end 174.645092 74.104908) (width 0.175) (layer B.Cu) (net 25))
-  (segment (start 167.227655 67.627655) (end 173.750931 67.627655) (width 0.175) (layer B.Cu) (net 25))
+  (segment (start 165.2 61.945481) (end 165.2 65.6) (width 0.175) (layer F.Cu) (net 25))
   (segment (start 173.750931 67.627655) (end 174.645092 68.521816) (width 0.175) (layer B.Cu) (net 25))
-  (segment (start 174.645092 74.104908) (end 173.099999 75.650001) (width 0.175) (layer B.Cu) (net 25))
+  (segment (start 164.914519 61.66) (end 165.2 61.945481) (width 0.175) (layer F.Cu) (net 25))
+  (segment (start 160.8 61.66) (end 164.914519 61.66) (width 0.175) (layer F.Cu) (net 25))
+  (via (at 165.2 65.6) (size 0.508) (drill 0.3302) (layers F.Cu B.Cu) (net 25))
   (segment (start 173.099999 75.650001) (end 172.25 76.5) (width 0.175) (layer B.Cu) (net 25))
-  (segment (start 165.2 62.218178) (end 165.2 65.6) (width 0.175) (layer F.Cu) (net 25))
-  (via (at 165.2 65.6) (size 0.508) (drill 0.3302) (layers F.Cu B.Cu) (net 25))
-  (segment (start 164.641822 61.66) (end 165.2 62.218178) (width 0.175) (layer F.Cu) (net 25))
-  (segment (start 160.8 61.66) (end 164.641822 61.66) (width 0.175) (layer F.Cu) (net 25))
   (segment (start 184 59.58) (end 182.806565 60.773435) (width 0.175) (layer B.Cu) (net 26))
   (segment (start 182.806565 60.773435) (end 165.773435 60.773435) (width 0.175) (layer B.Cu) (net 26))

Commit message: Ajustando PCBs
Signed-off-by: Gustavo Costa <gustavocosta@ic.ufal.br>
Parts:
- renumbered J6 to Anemometro, J1 to Biruta, J5 to Pluviometro, J2 to Power
Other:
- board text added: "+"
Changed lines of the file:
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@@
     (area 122.424999 49.924999 187.575001 110.075001)
     (thickness 1.6)
-    (drawings 14)
+    (drawings 15)
     (tracks 423)
     (zones 0)
@@
     (at 126.25 61.46 270)
     (descr "2-way 2.54mm pitch terminal block, Phoenix MPT series")
-    (fp_text reference J1 (at 1.27 -4.50088 360) (layer F.SilkS)
+    (fp_text reference Biruta (at 1.27 -4.75 360) (layer F.SilkS)
       (effects (font (size 0.5 0.5) (thickness 0.075)))
     )
@@
     (at 127.25 85.8 270)
     (descr "2-way 3.5mm pitch terminal block, Phoenix PT series")
-    (fp_text reference J2 (at 1.75 -4.3 360) (layer F.SilkS)
+    (fp_text reference Power (at 1.7 -4.75 360) (layer F.SilkS)
       (effects (font (size 0.5 0.5) (thickness 0.075)))
     )
@@
     (at 126.25 69.71 270)
     (descr "2-way 2.54mm pitch terminal block, Phoenix MPT series")
-    (fp_text reference J5 (at 1.27 -4.50088 360) (layer F.SilkS)
+    (fp_text reference Pluviometro (at 1.27 -5.75 360) (layer F.SilkS)
       (effects (font (size 0.5 0.5) (thickness 0.075)))
     )
@@
     (at 126.25 77.66 270)
     (descr "2-way 2.54mm pitch terminal block, Phoenix MPT series")
-    (fp_text reference J6 (at 1.27 -4.50088 360) (layer F.SilkS)
+    (fp_text reference Anemometro (at 1.27 -6 360) (layer F.SilkS)
       (effects (font (size 0.5 0.5) (thickness 0.075)))
     )
@@
     )
   )
+  (gr_text + (at 127.25 91.5) (layer F.SilkS)
+    (effects (font (size 0.5 0.5) (thickness 0.075)))
+  )
   (gr_arc (start 186.5 109) (end 187.5 109) (angle 90) (layer Edge.Cuts) (width 0.15))
