File: PCB - ESP devkit/Weather-Station.sch (KiCad schematic (older format))
At the start: 39 parts, among them J1 Biruta, J10 Conn_01x19, J11 Conn_01x19, J2 Power, J3 BH1750-FVI, J4 BME280, J5 Pluviometro, J6 Anemometro, J7 FTDI, J8 Conn_01x02, J9 Conn_01x02, SW1 SW_Push_SPDT, SW2 SW_Push, SW3 SW_SPDT, U1 AP1117-33

Commit message: Tirando o circuito de programação do ESP
Signed-off-by: Gustavo Costa <gustavocosta@ic.ufal.br>
Parts:
- removed J7: FTDI, Pin_Headers:Pin_Header_Straight_1x04_Pitch2.54mm, symbol Conn_01x04
- removed R16, R4, R6, R8: 10K, Resistors_SMD:R_0805, symbol R
- removed SW1: SW_Push_SPDT, Buttons_Switches_ThroughHole:SW_Micro_SPST, symbol SW_Push_SPDT
- removed SW3: SW_SPDT, Buttons_Switches_ThroughHole:SW_Micro_SPST, symbol SW_SPDT
Connections:
- net +3V3: now also C3.1, U1.2 (VO)
- net RXD: no longer names the net of J11.15 (Pin_15)
- net TXD: no longer names the net of J11.16 (Pin_16)
- no-connect marks 14 -> 19
Changed lines of the file:
@@
-$EndComp
-$Comp
-L Conn_01x04 J7
-U 1 1 5A5E7C94
-P 2000 2700
-F 0 "J7" H 2000 2900 50  0000 C CNN
-F 1 "FTDI" H 2000 2400 50  0000 C CNN
-F 2 "Pin_Headers:Pin_Header_Straight_1x04_Pitch2.54mm" H 2000 2700 50  0001 C CNN
-F 3 "" H 2000 2700 50  0001 C CNN
-	1    2000 2700
-	-1   0    0    1
-$EndComp
-$Comp
-L GND #PWR01
-U 1 1 5A5E7E47
-P 2250 2850
-F 0 "#PWR01" H 2250 2600 50  0001 C CNN
-F 1 "GND" H 2250 2700 50  0000 C CNN
-F 2 "" H 2250 2850 50  0001 C CNN
-F 3 "" H 2250 2850 50  0001 C CNN
-	1    2250 2850
-	1    0    0    -1
 $EndComp
 $Comp
@@
 $EndComp
 $Comp
-L R R4
-U 1 1 5A5E848D
-P 6450 4000
-F 0 "R4" V 6350 4000 50  0000 C CNN
-F 1 "10K" V 6450 4000 50  0000 C CNN
-F 2 "Resistors_SMD:R_0805" V 6380 4000 50  0001 C CNN
-F 3 "" H 6450 4000 50  0001 C CNN
-	1    6450 4000
-	1    0    0    -1
-$EndComp
-$Comp
 L SW_Push SW2
 U 1 1 5A5E86EC
@@
 $EndComp
 $Comp
-L R R6
-U 1 1 5A5E8FA0
-P 6550 4000
-F 0 "R6" V 6630 4000 50  0000 C CNN
-F 1 "10K" V 6550 4000 50  0000 C CNN
-F 2 "Resistors_SMD:R_0805" V 6480 4000 50  0001 C CNN
-F 3 "" H 6550 4000 50  0001 C CNN
-	1    6550 4000
-	1    0    0    -1
-$EndComp
-$Comp
 L R R7
 U 1 1 5A5E93FF
@@
 $EndComp
 $Comp
-L R R8
-U 1 1 5A5E9452
-P 7300 3900
-F 0 "R8" V 7380 3900 50  0000 C CNN
-F 1 "10K" V 7300 3900 50  0000 C CNN
-F 2 "Resistors_SMD:R_0805" V 7230 3900 50  0001 C CNN
-F 3 "" H 7300 3900 50  0001 C CNN
-	1    7300 3900
-	1    0    0    -1
-$EndComp
-$Comp
-L SW_Push_SPDT SW1
-U 1 1 5A5E955A
-P 3000 3050
-F 0 "SW1" H 3000 3220 50  0000 C CNN
-F 1 "SW_Push_SPDT" H 3000 2850 50  0000 C CNN
-F 2 "Buttons_Switches_ThroughHole:SW_Micro_SPST" H 3000 3050 50  0001 C CNN
-F 3 "" H 3000 3050 50  0001 C CNN
-	1    3000 3050
-	-1   0    0    1
-$EndComp
-Text GLabel 6300 2650 2    60   Input ~ 0
-TXD
-Text GLabel 6300 2750 2    60   Input ~ 0
-RXD
-Text GLabel 2300 2500 2    60   Input ~ 0
-TXD
-Text GLabel 2300 2600 2    60   Input ~ 0
-RXD
-$Comp
 L GND #PWR06
 U 1 1 5A5EAEB2
@@
 $EndComp
 $Comp
-L SW_SPDT SW3
-U 1 1 5AE74020
-P 7600 3650
-F 0 "SW3" H 7600 3820 50  0000 C CNN
-F 1 "SW_SPDT" H 7600 3450 50  0000 C CNN
-F 2 "Buttons_Switches_ThroughHole:SW_Micro_SPST" H 7600 3650 50  0001 C CNN
-F 3 "" H 7600 3650 50  0001 C CNN
-	1    7600 3650
-	1    0    0    -1
-$EndComp
-NoConn ~ 7800 3550
-$Comp
-L GND #PWR017
-U 1 1 5AE74368
-P 7850 3800
-F 0 "#PWR017" H 7850 3550 50  0001 C CNN
-F 1 "GND" H 7850 3650 50  0000 C CNN
-F 2 "" H 7850 3800 50  0001 C CNN
-F 3 "" H 7850 3800 50  0001 C CNN
-	1    7850 3800
-	1    0    0    -1
-$EndComp
-$Comp
-L GND #PWR018
-U 1 1 5AE786A0
-P 6550 4250
-F 0 "#PWR018" H 6550 4000 50  0001 C CNN
-F 1 "GND" H 6550 4100 50  0000 C CNN
-F 2 "" H 6550 4250 50  0001 C CNN
-F 3 "" H 6550 4250 50  0001 C CNN
-	1    6550 4250
-	1    0    0    -1
-$EndComp
-$Comp
 L R R11
 U 1 1 5AE78807
@@
 $EndComp
 Wire Wire Line
-	2200 2800 2250 2800
-Wire Wire Line
-	2250 2800 2250 2850
-Wire Wire Line
-	2200 2700 2600 2700
-Wire Wire Line
-	2600 2700 2600 2950
-Wire Wire Line
-	2600 2950 2800 2950
-Wire Wire Line
-	2450 3250 2650 3250
-Wire Wire Line
-	2650 3150 2650 3300
-Wire Wire Line
-	2650 3150 2800 3150
+	2450 3250 3200 3250
 Wire Wire Line
 	1450 3250 1850 3250
@@
 Connection ~ 4000 1600
 Wire Wire Line
-	2200 2500 2300 2500
-Wire Wire Line
-	2200 2600 2300 2600
-Wire Wire Line
-	1750 4800 7300 4800
-Wire Wire Line
 	6700 4250 10200 4250
 Wire Wire Line
@@
 Connection ~ 2150 3600
 Wire Wire Line
-	6300 3650 7400 3650
-Wire Wire Line
-	7300 3750 7300 3650
-Connection ~ 7300 3650
-Wire Wire Line
-	7800 3750 7850 3750
-Wire Wire Line
-	7850 3750 7850 3800
-Wire Wire Line
 	6300 3250 6400 3250
 Wire Wire Line
@@
 	7550 2850 6300 2850
 Wire Wire Line
-	6550 3750 6550 3850
-Wire Wire Line
-	7300 4800 7300 4050
-Connection ~ 3200 3050
-Wire Wire Line
-	6550 4150 6550 4250
-Wire Wire Line
 	4300 3800 4300 3850
 Wire Wire Line
@@
 Wire Wire Line
 	6300 2350 6500 2350
-Connection ~ 3200 4800
-Wire Wire Line
-	6700 3250 6700 4800
-Connection ~ 6700 4800
+Wire Wire Line
+	6700 4800 6700 3250
 Connection ~ 6700 3400
 Wire Wire Line
@@
 	1750 3300 1750 3250
 Connection ~ 1750 3250
-Connection ~ 2650 3250
 $Comp
 L GND #PWR022
@@
 	1750 4700 2550 4700
 Connection ~ 2150 4700
-$Comp
-L R R16
-U 1 1 5B2969BC
-P 4200 3600
-F 0 "R16" V 4100 3600 50  0000 C CNN
-F 1 "10K" V 4200 3600 50  0000 C CNN
-F 2 "Resistors_SMD:R_0805" V 4130 3600 50  0001 C CNN
-F 3 "" H 4200 3600 50  0001 C CNN
-	1    4200 3600
-	0    1    1    0
-$EndComp
-$Comp
-L GND #PWR026
-U 1 1 5B296AF3
-P 4000 3700
-F 0 "#PWR026" H 4000 3450 50  0001 C CNN
-F 1 "GND" H 4000 3550 50  0000 C CNN
-F 2 "" H 4000 3700 50  0001 C CNN
-F 3 "" H 4000 3700 50  0001 C CNN
-	1    4000 3700
-	1    0    0    -1
-$EndComp
-Wire Wire Line
-	4350 3600 4450 3600
-Wire Wire Line
-	4050 3600 4000 3600
-Wire Wire Line
-	4000 3600 4000 3700
 NoConn ~ 4450 3500
 $Comp
@@
 	1    0    0    -1
 $EndComp
+Wire Wire Line
+	4450 3700 4200 3700
+Wire Wire Line
+	4450 3800 4300 3800
+NoConn ~ 4450 3900
+NoConn ~ 4450 4000
+NoConn ~ 4450 4100
+NoConn ~ 4450 4200
+$Comp
+L GND #PWR027
+U 1 1 5B61D864
+P 6450 2950
+F 0 "#PWR027" H 6450 2700 50  0001 C CNN
+F 1 "GND" H 6450 2800 50  0000 C CNN
+F 2 "" H 6450 2950 50  0001 C CNN
+F 3 "" H 6450 2950 50  0001 C CNN
+	1    6450 2950
+	0    -1   -1   0
+$EndComp
+Wire Wire Line
+	6300 2950 6450 2950
+NoConn ~ 6300 3950
+NoConn ~ 6300 4050
+NoConn ~ 6300 4150
+Connection ~ 3200 3250
+Wire Wire Line
+	2650 3300 2650 3250
+Connection ~ 2650 3250
+NoConn ~ 6300 2650
+NoConn ~ 6300 2750
+NoConn ~ 4450 3600
+NoConn ~ 6300 3650
+NoConn ~ 6300 3750
 $Comp
 L Conn_01x19 J11
@@
 	-1   0    0    1
 $EndComp
-Wire Wire Line
-	4450 3700 4200 3700
-Wire Wire Line
-	4450 3800 4300 3800
-NoConn ~ 4450 3900
-NoConn ~ 4450 4000
-NoConn ~ 4450 4100
-NoConn ~ 4450 4200
-$Comp
-L GND #PWR027
-U 1 1 5B61D864
-P 6450 2950
-F 0 "#PWR027" H 6450 2700 50  0001 C CNN
-F 1 "GND" H 6450 2800 50  0000 C CNN
-F 2 "" H 6450 2950 50  0001 C CNN
-F 3 "" H 6450 2950 50  0001 C CNN
-	1    6450 2950
-	0    -1   -1   0
-$EndComp
-Wire Wire Line
-	6300 2950 6450 2950
-Wire Wire Line
-	6300 3750 6550 3750
-Wire Wire Line
-	6300 3850 6450 3850
-Wire Wire Line
-	6450 4150 6450 4800
-Connection ~ 6450 4800
-NoConn ~ 6300 3950
-NoConn ~ 6300 4050
-NoConn ~ 6300 4150
+NoConn ~ 6300 3850
+Wire Wire Line
+	1750 4800 6700 4800
+Connection ~ 3200 4800
 $EndSCHEMATC

Commit message: Feita a PCB com ESP32 devkit
Signed-off-by: Gustavo Costa <gustavocosta@ic.ufal.br>
Parts:
- removed C1: 100nF, Capacitors_SMD:C_0805, symbol C
- removed R5, R7: 10K, Resistors_SMD:R_0805, symbol R
- removed SW2: SW_Push, Buttons_Switches_THT:SW_PUSH_6mm, symbol SW_Push
Connections:
- no-connect marks 19 -> 21
Changed lines of the file:
@@
 $EndComp
 $Comp
-L GND #PWR02
+L GND #PWR01
 U 1 1 5A5E8030
 P 1500 3400
-F 0 "#PWR02" H 1500 3150 50  0001 C CNN
+F 0 "#PWR01" H 1500 3150 50  0001 C CNN
 F 1 "GND" H 1500 3250 50  0000 C CNN
 F 2 "" H 1500 3400 50  0001 C CNN
@@
 $EndComp
 $Comp
-L GND #PWR03
+L GND #PWR02
 U 1 1 5A5E805E
 P 2150 3650
-F 0 "#PWR03" H 2150 3400 50  0001 C CNN
+F 0 "#PWR02" H 2150 3400 50  0001 C CNN
 F 1 "GND" H 2150 3500 50  0000 C CNN
 F 2 "" H 2150 3650 50  0001 C CNN
@@
 $EndComp
 $Comp
-L GND #PWR04
+L GND #PWR03
 U 1 1 5A5E841F
 P 2150 4300
-F 0 "#PWR04" H 2150 4050 50  0001 C CNN
+F 0 "#PWR03" H 2150 4050 50  0001 C CNN
 F 1 "GND" H 2150 4150 50  0000 C CNN
 F 2 "" H 2150 4300 50  0001 C CNN
@@
 $EndComp
 $Comp
-L SW_Push SW2
-U 1 1 5A5E86EC
-P 3900 1850
-F 0 "SW2" H 3950 1950 50  0000 L CNN
-F 1 "SW_Push" H 3900 1790 50  0000 C CNN
-F 2 "Buttons_Switches_THT:SW_PUSH_6mm" H 3900 2050 50  0001 C CNN
-F 3 "" H 3900 2050 50  0001 C CNN
-	1    3900 1850
-	0    -1   -1   0
-$EndComp
-$Comp
-L C C1
-U 1 1 5A5E875B
-P 4150 1850
-F 0 "C1" H 4175 1950 50  0000 L CNN
-F 1 "100nF" H 4175 1750 50  0000 L CNN
-F 2 "Capacitors_SMD:C_0805" H 4188 1700 50  0001 C CNN
-F 3 "" H 4150 1850 50  0001 C CNN
-	1    4150 1850
-	1    0    0    -1
-$EndComp
-$Comp
-L GND #PWR05
-U 1 1 5A5E8828
-P 4000 1550
-F 0 "#PWR05" H 4000 1300 50  0001 C CNN
-F 1 "GND" H 4000 1400 50  0000 C CNN
-F 2 "" H 4000 1550 50  0001 C CNN
-F 3 "" H 4000 1550 50  0001 C CNN
-	1    4000 1550
-	-1   0    0    1
-$EndComp
-$Comp
-L R R5
-U 1 1 5A5E8BF7
-P 3700 2500
-F 0 "R5" V 3780 2500 50  0000 C CNN
-F 1 "10K" V 3700 2500 50  0000 C CNN
-F 2 "Resistors_SMD:R_0805" V 3630 2500 50  0001 C CNN
-F 3 "" H 3700 2500 50  0001 C CNN
-	1    3700 2500
-	0    1    1    0
-$EndComp
-$Comp
-L R R7
-U 1 1 5A5E93FF
-P 6550 3250
-F 0 "R7" V 6630 3250 50  0000 C CNN
-F 1 "10K" V 6550 3250 50  0000 C CNN
-F 2 "Resistors_SMD:R_0805" V 6480 3250 50  0001 C CNN
-F 3 "" H 6550 3250 50  0001 C CNN
-	1    6550 3250
-	0    1    1    0
-$EndComp
-$Comp
-L GND #PWR06
+L GND #PWR04
 U 1 1 5A5EAEB2
 P 10450 3850
-F 0 "#PWR06" H 10450 3600 50  0001 C CNN
+F 0 "#PWR04" H 10450 3600 50  0001 C CNN
 F 1 "GND" H 10450 3700 50  0000 C CNN
 F 2 "" H 10450 3850 50  0001 C CNN
@@
 $EndComp
 $Comp
-L GND #PWR07
+L GND #PWR05
 U 1 1 5A5EAEF0
 P 9800 2550
-F 0 "#PWR07" H 9800 2300 50  0001 C CNN
+F 0 "#PWR05" H 9800 2300 50  0001 C CNN
 F 1 "GND" H 9800 2400 50  0000 C CNN
 F 2 "" H 9800 2550 50  0001 C CNN
@@
 $EndComp
 $Comp
-L +3.3V #PWR08
+L +3.3V #PWR06
 U 1 1 5A5EB03C
 P 3200 2350
-F 0 "#PWR08" H 3200 2200 50  0001 C CNN
+F 0 "#PWR06" H 3200 2200 50  0001 C CNN
 F 1 "+3.3V" H 3200 2490 50  0000 C CNN
 F 2 "" H 3200 2350 50  0001 C CNN
@@
 NoConn ~ 7650 1600
 $Comp
-L GND #PWR09
+L GND #PWR07
 U 1 1 5A5EB757
 P 7750 1700
-F 0 "#PWR09" H 7750 1450 50  0001 C CNN
+F 0 "#PWR07" H 7750 1450 50  0001 C CNN
 F 1 "GND" H 7750 1550 50  0000 C CNN
 F 2 "" H 7750 1700 50  0001 C CNN
@@
 $EndComp
 $Comp
-L +3.3V #PWR010
+L +3.3V #PWR08
 U 1 1 5A5EB998
 P 7350 1700
-F 0 "#PWR010" H 7350 1550 50  0001 C CNN
+F 0 "#PWR08" H 7350 1550 50  0001 C CNN
 F 1 "+3.3V" H 7350 1840 50  0000 C CNN
 F 2 "" H 7350 1700 50  0001 C CNN
@@
 $EndComp
 $Comp
-L +3.3V #PWR011
+L +3.3V #PWR09
 U 1 1 5A5EBA4C
 P 7950 1700
-F 0 "#PWR011" H 7950 1550 50  0001 C CNN
+F 0 "#PWR09" H 7950 1550 50  0001 C CNN
 F 1 "+3.3V" H 7950 1840 50  0000 C CNN
 F 2 "" H 7950 1700 50  0001 C CNN
@@
 $EndComp
 $Comp
-L GND #PWR012
+L GND #PWR010
 U 1 1 5A5EBA8A
 P 8150 1700
-F 0 "#PWR012" H 8150 1450 50  0001 C CNN
+F 0 "#PWR010" H 8150 1450 50  0001 C CNN
 F 1 "GND" H 8150 1550 50  0000 C CNN
 F 2 "" H 8150 1700 50  0001 C CNN
@@
 $EndComp
 $Comp
-L +3.3V #PWR013
+L +3.3V #PWR011
 U 1 1 5A5EBAC8
 P 8500 2100
-F 0 "#PWR013" H 8500 1950 50  0001 C CNN
+F 0 "#PWR011" H 8500 1950 50  0001 C CNN
 F 1 "+3.3V" H 8500 2240 50  0000 C CNN
 F 2 "" H 8500 2100 50  0001 C CNN
@@
 $EndComp
 $Comp
-L PWR_FLAG #FLG014
+L PWR_FLAG #FLG012
 U 1 1 5A5EBFFB
 P 1550 3200
-F 0 "#FLG014" H 1550 3275 50  0001 C CNN
+F 0 "#FLG012" H 1550 3275 50  0001 C CNN
 F 1 "PWR_FLAG" H 1550 3350 50  0000 C CNN
 F 2 "" H 1550 3200 50  0001 C CNN
@@
 $EndComp
 $Comp
-L PWR_FLAG #FLG015
+L PWR_FLAG #FLG013
 U 1 1 5A5EC039
 P 3150 2650
-F 0 "#FLG015" H 3150 2725 50  0001 C CNN
+F 0 "#FLG013" H 3150 2725 50  0001 C CNN
 F 1 "PWR_FLAG" H 3150 2800 50  0000 C CNN
 F 2 "" H 3150 2650 50  0001 C CNN
@@
 $EndComp
 $Comp
-L PWR_FLAG #FLG016
+L PWR_FLAG #FLG014
 U 1 1 5A5EC134
 P 2300 3600
-F 0 "#FLG016" H 2300 3675 50  0001 C CNN
+F 0 "#FLG014" H 2300 3675 50  0001 C CNN
 F 1 "PWR_FLAG" H 2300 3750 50  0000 C CNN
 F 2 "" H 2300 3600 50  0001 C CNN
@@
 $EndComp
 $Comp
-L GND #PWR019
+L GND #PWR015
 U 1 1 5AE78B79
 P 3900 4300
-F 0 "#PWR019" H 3900 4050 50  0001 C CNN
+F 0 "#PWR015" H 3900 4050 50  0001 C CNN
 F 1 "GND" H 3900 4150 50  0000 C CNN
 F 2 "" H 3900 4300 50  0001 C CNN
@@
 $EndComp
 $Comp
-L GND #PWR020
+L GND #PWR016
 U 1 1 5AE78CB9
 P 6500 2350
-F 0 "#PWR020" H 6500 2100 50  0001 C CNN
+F 0 "#PWR016" H 6500 2100 50  0001 C CNN
 F 1 "GND" H 6500 2200 50  0000 C CNN
 F 2 "" H 6500 2350 50  0001 C CNN
@@
 $EndComp
 $Comp
-L GND #PWR021
+L GND #PWR017
 U 1 1 5AE78F28
 P 4200 3700
-F 0 "#PWR021" H 4200 3450 50  0001 C CNN
+F 0 "#PWR017" H 4200 3450 50  0001 C CNN
 F 1 "GND" H 4200 3550 50  0000 C CNN
 F 2 "" H 4200 3700 50  0001 C CNN
@@
 	2150 4400 2150 4300
 Wire Wire Line
-	4000 2050 4000 2500
-Wire Wire Line
-	3900 2050 4150 2050
-Wire Wire Line
-	4150 2050 4150 2000
-Connection ~ 4000 2050
-Wire Wire Line
-	3900 1650 3900 1600
-Wire Wire Line
-	3900 1600 4150 1600
-Wire Wire Line
-	4150 1600 4150 1700
-Wire Wire Line
-	4000 1550 4000 1600
-Connection ~ 4000 1600
-Wire Wire Line
 	6700 4250 10200 4250
 Wire Wire Line
@@
 Connection ~ 2150 3600
 Wire Wire Line
-	6300 3250 6400 3250
-Wire Wire Line
-	3850 2500 4450 2500
-Connection ~ 4000 2500
-Wire Wire Line
-	3200 2500 3550 2500
-Wire Wire Line
 	4450 2400 3200 2400
-Connection ~ 3200 2500
 Wire Wire Line
 	7450 2550 6300 2550
@@
 Wire Wire Line
 	6300 2350 6500 2350
-Wire Wire Line
-	6700 4800 6700 3250
-Connection ~ 6700 3400
 Wire Wire Line
 	9800 2950 9800 3050
@@
 Connection ~ 1750 3250
 $Comp
-L GND #PWR022
+L GND #PWR018
 U 1 1 5AE7D2C5
 P 2650 3600
-F 0 "#PWR022" H 2650 3350 50  0001 C CNN
+F 0 "#PWR018" H 2650 3350 50  0001 C CNN
 F 1 "GND" H 2650 3450 50  0000 C CNN
 F 2 "" H 2650 3600 50  0001 C CNN
@@
 $EndComp
 $Comp
-L GND #PWR023
+L GND #PWR019
 U 1 1 5AE7D30B
 P 1750 3600
-F 0 "#PWR023" H 1750 3350 50  0001 C CNN
+F 0 "#PWR019" H 1750 3350 50  0001 C CNN
 F 1 "GND" H 1750 3450 50  0000 C CNN
 F 2 "" H 1750 3600 50  0001 C CNN
@@
 	4950 6850 4950 6650
 $Comp
-L GND #PWR024
+L GND #PWR020
 U 1 1 5AE9E1A8
 P 4500 6950
-F 0 "#PWR024" H 4500 6700 50  0001 C CNN
+F 0 "#PWR020" H 4500 6700 50  0001 C CNN
 F 1 "GND" H 4500 6800 50  0000 C CNN
 F 2 "" H 4500 6950 50  0001 C CNN
@@
 Connection ~ 6300 6250
 $Comp
-L GND #PWR025
+L GND #PWR021
 U 1 1 5AEA02F5
 P 6100 6950
-F 0 "#PWR025" H 6100 6700 50  0001 C CNN
+F 0 "#PWR021" H 6100 6700 50  0001 C CNN
 F 1 "GND" H 6100 6800 50  0000 C CNN
 F 2 "" H 6100 6950 50  0001 C CNN
@@
 NoConn ~ 4450 4200
 $Comp
-L GND #PWR027
+L GND #PWR022
 U 1 1 5B61D864
 P 6450 2950
-F 0 "#PWR027" H 6450 2700 50  0001 C CNN
+F 0 "#PWR022" H 6450 2700 50  0001 C CNN
 F 1 "GND" H 6450 2800 50  0000 C CNN
 F 2 "" H 6450 2950 50  0001 C CNN
@@
 NoConn ~ 6300 3850
 Wire Wire Line
-	1750 4800 6700 4800
+	6700 4800 1750 4800
 Connection ~ 3200 4800
+NoConn ~ 4450 2500
+Wire Wire Line
+	6700 3400 6700 4800
+NoConn ~ 6300 3250
 $EndSCHEMATC

Commit message: Ajustando PCBs
Signed-off-by: Gustavo Costa <gustavocosta@ic.ufal.br>
Parts:
- removed D1, D2, D4, D5: D, Diodes_SMD:D_SOD-123, symbol D
- removed J10, J11: Conn_01x19, Pin_Headers:Pin_Header_Straight_1x19_Pitch2.54mm, symbol Conn_01x19
- removed J3: BH1750-FVI, TerminalBlock_Phoenix:TerminalBlock_Phoenix_MPT-2.54mm_5pol, symbol Conn_01x05
- removed R12, R13: 1.5K, Resistors_SMD:R_0805, symbol R
- added C4, C5: 22μF, Capacitors_SMD:CP_Elec_6.3x7.7, symbol CP1
- added C6, C7, C8, C9: 0.1uF, Capacitors_SMD:C_0805, symbol C
- added J10, J11, J12, J13, J14, J15: Conn_01x02, TerminalBlock_Phoenix:TerminalBlock_Phoenix_MPT-2.54mm_2pol, symbol Conn_01x02
- added J16, J7: Conn_01x19, Pin_Headers:Pin_Header_Straight_1x19_Pitch2.54mm, symbol Conn_01x19
- added J3: DataLogger, Pin_Headers:Pin_Header_Straight_1x08_Pitch2.54mm, symbol Conn_01x08
- added U3: AP1117-33, TO_SOT_Packages_SMD:SOT-223, symbol AP1117-33
- added U4, U5, U6, U7: ADS1115, Housings_SSOP:MSOP-10_3x3mm_Pitch0.5mm, symbol ADS1115
- J2: footprint TerminalBlock_Phoenix:TerminalBlock_Phoenix_MPT-2.54mm_2pol -> TerminalBlock_Phoenix:TerminalBlock_Phoenix_PT-3.5mm_2pol
- R10, R9: value 1.5K -> 10k
Connections:
- net +3V3: now also J7.1 (Pin_1)
- net GND: now also C4.2, C5.2, C6.2, C7.2, C8.2, C9.2, J16.1 (Pin_1), J16.7 (Pin_7), J3.7 (Pin_7), J7.14 (Pin_14), U3.1 (GND), U4.1 (ADDR), U4.3 (GND), U5.3 (GND), U6.3 (GND), U7.3 (GND); no longer R10.2, R9.2
- net at J6.1 (Pin_1), R3.1: now also J7.9 (Pin_9)
- net at J5.1 (Pin_1), R2.2: now also J7.8 (Pin_8)
- net SCL: now reaches J4.3 (Pin_3)
- net SCL: now also R9.2, J16.3 (Pin_3), J3.5 (Pin_5), U4.10 (SCL), U5.10 (SCL), U6.1 (ADDR), U6.10 (SCL), U7.10 (SCL)
- net SDA: now reaches J4.4 (Pin_4)
- net SDA: now also R10.2, J16.6 (Pin_6), J3.6 (Pin_6), U4.9 (SDA), U5.9 (SDA), U6.9 (SDA), U7.1 (ADDR), U7.9 (SDA)
- net at C2.1, J2.2 (Pin_2), U1.3 (VI): now also C4.1, U3.3 (VI)
- net at R11.1: now also J7.15 (Pin_15)
- net ADC1_CH0: no longer names the net of J8.1 (Pin_1)
- net ADC1_CH0: now also U4.4 (AIN0); no longer R9.1
- net ADC1_CH3: no longer names the net of J8.2 (Pin_2)
- net ADC1_CH3: now also U4.5 (AIN1); no longer R10.1
- net ADC1_CH4: no longer names the net of J1.2 (Pin_2), R1.1
- net ADC1_CH4: now also J7.7 (Pin_7)
- net ADC1_CH6: no longer names the net of J9.1 (Pin_1)
- net ADC1_CH6: now also U4.6 (AIN2)
- net ADC1_CH7: no longer names the net of J9.2 (Pin_2)
- net ADC1_CH7: now also U4.7 (AIN3)
- new net: J10.1 (Pin_1), U5.4 (AIN0)
- new net: J10.2 (Pin_2), U5.5 (AIN1)
- new net: J11.1 (Pin_1), U5.6 (AIN2)
- new net: J11.2 (Pin_2), U5.7 (AIN3)
- new net: J12.1 (Pin_1), U6.4 (AIN0)
- new net: J12.2 (Pin_2), U6.5 (AIN1)
- new net: J13.1 (Pin_1), U6.6 (AIN2)
- new net: J13.2 (Pin_2), U6.7 (AIN3)
- new net: J14.1 (Pin_1), U7.4 (AIN0)
- new net: J14.2 (Pin_2), U7.5 (AIN1)
- new net: J15.1 (Pin_1), U7.6 (AIN2)
- new net: J15.2 (Pin_2), U7.7 (AIN3)
- new net +5V: C5.1, C6.1, C7.1, C8.1, C9.1, J3.8 (Pin_8), R10.1, R9.1, U3.2 (VO), U4.8 (VDD), U5.1 (ADDR), U5.8 (VDD), U6.8 (VDD), U7.8 (VDD)
- new net CS: J16.11 (Pin_11), J3.1 (Pin_1)
- new net MISO: J16.8 (Pin_8), J3.3 (Pin_3)
- new net MOSI: J16.2 (Pin_2), J3.2 (Pin_2)
- new net SCK: J16.9 (Pin_9), J3.4 (Pin_4)
- no-connect marks 21 -> 28
Other:
- moved on the sheet: C2, C3, D3, J1, J2, J4, J5, J6, R1, R11, R14, R15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
